Commit message: Task4A and 4B done

File: MiniTask/src/minitask/urdf/tuktuk.urdf (robot description, URDF)
Before this commit: robot tuktuk, 18 links, 17 joints
Links:
- added link dummy_link1
- added link dummy_link2
- added link irl; visual box size=0.1 0.1 0.1
- added link irr; visual box size=0.1 0.1 0.1
Joints:
- removed joint ball_n_socket
- added joint ball_n_socketx: type continuous, parent caster_stud, child dummy_link1, origin xyz=0 0 -0.04 rpy=0 0 0, axis 1 0 0
- added joint ball_n_sockety: type continuous, parent dummy_link1, child dummy_link2, origin xyz=0 0 0 rpy=0 0 0, axis 0 1 0
- added joint ball_n_socketz: type continuous, parent dummy_link2, child caster_ball, origin xyz=0 0 0 rpy=0 0 0, axis 0 0 1
- added joint irl_joint: type fixed, parent chassis, child irl, origin xyz=0.3 0.25 0.08 rpy=0 0 0
- added joint irr_joint: type fixed, parent chassis, child irr, origin xyz=0.3 -0.25 0.08 rpy=0 0 0
- joint iwheel1_joint: axis (none) -> 0 0 1; type fixed -> continuous
- joint iwheel2_joint: axis (none) -> 0 0 1; type fixed -> continuous
- joint wheel1_joint: origin xyz=0 -0.125 0 rpy=1.57 0 0 -> xyz=0 0 0 rpy=0 0 0; parent motor1 -> iwheel1
- joint wheel2_joint: origin xyz=0 0.125 0 rpy=1.57 0 0 -> xyz=0 0 0 rpy=0 0 0; parent motor2 -> iwheel2
