Commit message: Inertial Edit

File: Task4/src/task4/urdf/macros.xacro (robot description, xacro)
@@ -2,28 +2,56 @@
 <robot xmlns:xacro="http://www.ros.org/wiki/xacro">
     <!-- Def Inertial -->
-    <xacro:macro name="default_inertial" params="mass">
+    <xacro:macro name="box_inertial" params="mass x y z">
         <inertial>
             <mass value="${mass}"/>
             <origin xyz="0 0 0" rpy="0 0 0"/>
             <inertia
-                ixx="${mass*0.001}"
+                ixx="${mass*(y*y + z*z)/12}"
                 ixy="0"
                 ixz="0"
-                iyy="${mass*0.001}"
+                iyy="${mass*(x*x + z*z)/12}"
                 iyz="0"
-                izz="${mass*0.001}"/>
+                izz="${mass*(x*x + y*y)/12}"/>
+        </inertial>
+    </xacro:macro>
+    <xacro:macro name="cylinder_inertial"
+             params="mass radius length">
+        <inertial>
+            <mass value="${mass}"/>
+            <origin xyz="0 0 0" rpy="0 0 0"/>
+            <inertia
+                ixx="${mass*(3*radius*radius + length*length)/12}"
+                ixy="0"
+                ixz="0"
+                iyy="${mass*(3*radius*radius + length*length)/12}"
+                iyz="0"
+                izz="${mass*radius*radius/2}"/>
+        </inertial>
+    </xacro:macro>
+    <xacro:macro name="sphere_inertial"
+             params="mass radius">
+        <inertial>
+            <mass value="${mass}"/>
+            <origin xyz="0 0 0" rpy="0 0 0"/>
+            <inertia
+                ixx="${2*mass*radius*radius/5}"
+                ixy="0"
+                ixz="0"
+                iyy="${2*mass*radius*radius/5}"
+                iyz="0"
+                izz="${2*mass*radius*radius/5}"/>
         </inertial>
     </xacro:macro>
     <xacro:macro name="zero_inertial">
         <inertial>
-            <mass value="0"/>
+            <mass value="0.001"/>
             <origin xyz="0 0 0" rpy="0 0 0"/>
             <inertia
-                ixx="0"
+                ixx="0.001"
                 ixy="0"
                 ixz="0"
-                iyy="0"
+                iyy="0.001"
                 iyz="0"
-                izz="0"/>
+                izz="0.001"/>
         </inertial>
     </xacro:macro>
@@ -31,5 +59,8 @@
     <xacro:macro name="ir_module" params="name x y z">
         <link name="${name}">
-            <xacro:default_inertial mass="${ir_mass}"/>
+            <xacro:box_inertial mass="${ir_mass}"
+                                x="${ir_size}"
+                                y="${ir_size}"
+                                z="${ir_size}"/>
             <visual>
                 <geometry>
@@ -53,5 +84,8 @@
     <xacro:macro name="drive_side" params="side motor_y wheel_y">
         <link name="motor${side}">
-            <xacro:default_inertial mass="${motor_mass}"/>
+            <xacro:box_inertial mass="${motor_mass}"
+                                x="${motor_l}"
+                                y="${motor_w}"
+                                z="${motor_h}"/>
             <visual>
                 <geometry>
@@ -72,5 +106,7 @@
         </joint>
         <link name="iwheel${side}">
-            <xacro:default_inertial mass="${iwheel_mass}"/>
+            <xacro:cylinder_inertial mass="${iwheel_mass}"
+                                     radius="${iwheel_r}"
+                                     length="${wheel_w}"/>
             <visual>
                 <geometry>
@@ -92,5 +128,7 @@
         </joint>
         <link name="wheel${side}">
-            <xacro:default_inertial mass="${wheel_mass}"/>
+            <xacro:cylinder_inertial mass="${wheel_mass}"
+                                     radius="${wheel_r}"
+                                     length="${wheel_w}"/>
             <visual>
                 <geometry>
@@ -114,8 +152,10 @@
     <xacro:macro name="caster_assembly">
         <link name="caster_base">
-            <xacro:default_inertial mass="${caster_base_mass}"/>
-            <visual>
-                <geometry>
-                    <box size="${caster_base_size} ${caster_base_size} ${caster_base_h}"/>
+            <xacro:cylinder_inertial mass="${caster_base_mass}"
+                                     radius="${caster_base_r}"
+                                     length="${caster_base_w}"/>
+            <visual>
+                <geometry>
+                    <cylinder radius="${caster_base_r}" length="${caster_base_w}" />
                 </geometry>
                 <material name="red"/>
@@ -123,5 +163,5 @@
             <collision>
                 <geometry>
-                    <box size="${caster_base_size} ${caster_base_size} ${caster_base_h}"/>
+                    <cylinder radius="${caster_base_r}" length="${caster_base_w}" />
                 </geometry>
             </collision>
@@ -133,5 +173,7 @@
         </joint>
         <link name="caster_stud">
-            <xacro:default_inertial mass="${caster_stud_mass}"/>
+            <xacro:cylinder_inertial mass="${caster_stud_mass}"
+                                     radius="${caster_stud_r}"
+                                     length="${caster_stud_h}"/>
             <visual>
                 <geometry>
@@ -152,5 +194,5 @@
         </joint>
         <link name="dummy_link1">
-            <xacro:default_inertial mass="${caster_stud_mass}"/>
+            <xacro:zero_inertial />
             <collision >
                 <geometry>
@@ -160,5 +202,5 @@
         </link>
         <link name="dummy_link2">
-            <xacro:default_inertial mass="${caster_stud_mass}"/>
+            <xacro:zero_inertial />
             <collision >
                 <geometry>
@@ -168,5 +210,6 @@
         </link>
         <link name="caster_ball">
-            <xacro:default_inertial mass="${caster_ball_mass}"/>
+            <xacro:sphere_inertial mass="${caster_ball_mass}"
+                                     radius="${caster_ball_r}"/>
             <visual>
                 <geometry>
@@ -203,5 +246,8 @@
     <xacro:macro name="controller_assembly" params="name mat y_offset z_offset">
         <link name="${name}">
-            <xacro:default_inertial mass="${controller_mass}"/>
+            <xacro:box_inertial mass="${controller_mass}"
+                                x="${controller_side}"
+                                y="${controller_side}"
+                                z="${controller_h}"/>
             <visual>
                 <geometry>
@@ -225,5 +271,8 @@
     <xacro:macro name="battery">
         <link name="battery">
-            <xacro:default_inertial mass="${battery_mass}"/>
+            <xacro:box_inertial mass="${battery_mass}"
+                                x="${battery_l}"
+                                y="${battery_w}"
+                                z="${battery_h}"/>
             <visual>
                 <geometry>
@@ -246,5 +295,7 @@
     <xacro:macro name="switch">
         <link name="switch">
-            <xacro:default_inertial mass="${switch_mass}"/>
+            <xacro:cylinder_inertial mass="${switch_mass}"
+                                     radius="${switch_r}"
+                                     length="${switch_w}"/>
             <visual>
                 <geometry>
@@ -286,12 +337,13 @@
     </xacro:macro>
 </robot>
-<!-- there are only 2 types of inertials used here default and zero
- default is used in every link and zero in dummy links
- the default inertials use only ixx iyy and izz and mass for rough calculations.
- arduino driver motors IRs battery and switch serve no purpose. they are only there for visual effects
+<!-- There are only 4 types of inertials used here box, cylinder, sphere and zero.
+ Zero has negligible values and are used in dummy links
+ Box, cylinder and sphere use the moment of inertia aboutt respective axes of cuboid, cylinder and sphere respectively.
+ Only MI about xx, yy,zz are considered (for ideal result).
+ Arduino, driver, motors, IRs, battery and switch serve no purpose. They are only there for visual effects
  IR 1-4 are the front IRs of the linebot
  IR l and r  are the IRs that detected the obstacles in line bot path
- task mentions to join drive wheels to chassis but i connected drive wheels to motor so that if i move the motors, drive wheels will go with it
- drive wheels consist of 2 cylinders iwheel (yellow) which actually moves and wheel (blacK) whihc is a tyre.
- between caster_stud and caster_ball there are 2 dummy links to enable ball and socket type motion:
+ Task-4 mentions to join drive wheels to chassis but I connected drive wheels to motor so that if I move the motors, drive wheels will go with it.
+ Drive wheels consist of 2 cylinders iwheel (yellow) which actually moves and wheel (blacK) whihc is like a tyre.
+ Between caster_stud and caster_ball there are 2 dummy links to enable ball and socket type motion:
     stud to link1: continuous joint in x dir, link1 to link2: cont joint in y dir and then link2 to ball: cont joint in z dir-->

File: Task4/src/task4/urdf/properties.xacro (robot description, xacro)
@@ -43,6 +43,6 @@
     <xacro:property name="ir_size" value="0.1"/>
     <!-- Caster -->
-    <xacro:property name="caster_base_size" value="0.1"/>
-    <xacro:property name="caster_base_h" value="0.05"/>
+    <xacro:property name="caster_base_r" value="0.08"/>
+    <xacro:property name="caster_base_w" value="0.05"/>
     <xacro:property name="caster_stud_r" value="0.025"/>
     <xacro:property name="caster_stud_h" value="0.08"/>

File: Task4/src/task4/urdf/tuktuk.urdf (robot description, URDF)
Before this commit: robot tuktuk, 22 links, 21 joints
Links:
- link caster_base: geometry collision cylinder length=0.05 radius=0.08; visual cylinder length=0.05 radius=0.08
- link dummy_link1: mass 0.01 -> 0.001
- link dummy_link2: mass 0.01 -> 0.001

File: Task4/src/task4/urdf/tuktuk.xacro (robot description, xacro)
@@ -6,5 +6,8 @@
     <xacro:include filename="gazebo.xacro"/>
     <link name="chassis">
-        <xacro:default_inertial mass="${chassis_mass}"/>
+        <xacro:box_inertial mass="${chassis_mass}"
+                            x="${chassis_l}"
+                            y="${chassis_w}"
+                            z="${chassis_h}"/>
         <visual>
             <geometry>
@@ -21,12 +24,12 @@
     <xacro:main_assembly/>
 </robot>
-<!-- I used xacro to make this bot coz its easy to modify this way
-    most of the dimensions and origin of links are in properties.xacro
-    macros.xacro has all the macros used in main_assembly macro itself
-    materials.xacro has the colors(materials)
-    gazebo.xacro has the diff drive plugin used in task 4b
-    i used chassis instead of base_link
-    the original tuktuk is in MiniTask
-    more logic is inside macros.xacro
-    KDL might throw a warning coz kdl does not support root link with inertia
+<!-- I used xacro to make this bot coz its easy to modify this way.
+    Most of the dimensions and origin of links are in properties.xacro.
+    macros.xacro has all the macros used in main_assembly macro itself.
+    materials.xacro has the colors(materials).
+    gazebo.xacro has the diff drive plugin used in task 4b.
+    I used chassis instead of base_link.
+    The original tuktuk is in MiniTask.
+    More logic is inside macros.xacro
+    KDL might throw a warning coz kdl does not support root link with inertia,
     but i did not create a dummy link coz without inertial and collision, chassis will be invisible in gazebo-->
